File: final_project/Electrical/final_project/final_project.kicad_pcb (KiCad board)
At the start: 2 copper layers, 1 part, among them J1 Raspberry_Pi_4b

Commit message: Top plate v7, gripper v1, electrical v1
Parts:
- added J2: Back_Right_Encoder, Connector_PinHeader_1.00mm:PinHeader_1x03_P1.00mm_Vertical, F.Cu at (152.4, 78.7)
- added J3: Servo, Connector_PinHeader_1.00mm:PinHeader_1x03_P1.00mm_Vertical, F.Cu at (152.4, 66.0)
- added J7: Front_Left_Encoder, Connector_PinHeader_1.00mm:PinHeader_1x03_P1.00mm_Vertical, F.Cu at (144.8, 78.7)
- added J8: Ultrasonic, Connector_PinHeader_1.00mm:PinHeader_1x04_P1.00mm_Vertical, F.Cu at (147.3, 66.0)
- added J9: H-Bridge, Connector_PinHeader_1.00mm:PinHeader_1x04_P1.00mm_Vertical, F.Cu at (149.9, 76.2)
- added R1: 1k, Resistor_SMD:R_0201_0603Metric, F.Cu at (139.7, 68.6)
- added R2: 2k, Resistor_SMD:R_0201_0603Metric, F.Cu at (141.9, 71.1)
- moved J1 120.9 mm to (136.2, 63.5)
Routing:
- net /GND: track 0.00 -> 45.0 mm
- net /3.3V: track 0.00 -> 31.5 mm
- net /FLENC: track 0.00 -> 30.4 mm
- net /Servo: track 0.00 -> 23.2 mm
- net /TRIG: track 0.00 -> 16.2 mm
- net /5v: track 0.00 -> 12.5 mm
- net Net-(J8-Pin_3): track 0.00 -> 11.1 mm
- net /ECHO: track 0.00 -> 7.07 mm
