File: final_project/Electrical/final_project/final_project.kicad_sch (KiCad schematic)
At the start: 11 parts, among them J1 Raspberry_Pi_4b, J2 Back_Right_Encoder, J3 Servo, J4 Left_Motors, J5 Right_Motors, J6 H-Bridge_Power, J7 Front_Left_Encoder, J8 Ultrasonic, J9 H-Bridge

Commit message: Top plate v7, gripper v1, electrical v1
Parts:
- R2: footprint (none) -> Resistor_SMD:R_0201_0603Metric
Changed lines of the file:
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@@
       (effects (font (size 1.27 1.27)) (justify left))
     )
-    (property "Footprint" "" (at 65.532 53.34 90)
+    (property "Footprint" "Resistor_SMD:R_0201_0603Metric" (at 65.532 53.34 90)
       (effects (font (size 1.27 1.27)) hide)
     )
